Commit message: Add files via upload

File: car_model_description/urdf/car_model.urdf (robot description, URDF)
Before this commit: robot car_model, 11 links, 10 joints
Links:
- link base_link: geometry collision box size=1.8 1.2 0.2; visual box size=1.8 1.2 0.2
Joints:
- joint hokuyo_joint: origin xyz=1.5 0 -0.5 rpy=0 0 0 -> xyz=2.1 0 -0.5 rpy=0 0 0
- joint left_front_wheel_joint: origin xyz=0 0.1 -0.1 rpy=0 0 0 -> xyz=0 -0.1 -0.1 rpy=0 0 0
- joint left_rear_wheel_joint: origin xyz=-1.1 -0.8 -0.3 rpy=0 0 0 -> xyz=0 -0.7 -0.3 rpy=0 0 0
- joint left_steer_joint: origin xyz=1.2 -0.8 -0.25 rpy=0 0 0 -> xyz=1.8 -0.5 -0.25 rpy=0 0 0
- joint rear_wheel_joint: origin xyz=-1.2 0 -0.25 rpy=0 0 0 -> xyz=0 0 -0.25 rpy=0 0 0
- joint right_rear_wheel_joint: origin xyz=-1.1 0.8 -0.3 rpy=0 0 0 -> xyz=0 0.7 -0.3 rpy=0 0 0
- joint right_steer_joint: origin xyz=1.2 0.8 -0.25 rpy=0 0 0 -> xyz=1.8 0.5 -0.25 rpy=0 0 0
- joint steer_joint: origin xyz=1.2 0 -0.25 rpy=0 0 0 -> xyz=1.8 0 -0.25 rpy=0 0 0

Commit message: Add files via upload

File: car_model_description/urdf/car_model.urdf (robot description, URDF)
Before this commit: robot car_model, 11 links, 10 joints
Links:
- link base_link: geometry collision mesh filename=package://car_model_description/meshes/whole_car.stl scale=0.001 0.001 0.001; visual mesh filename=package://car_model_description/meshes/whole_car.stl scale=0.001 0.001 0.001
Joints:
- joint hokuyo_joint: origin xyz=2.1 0 -0.5 rpy=0 0 0 -> xyz=2.4 0.5 -0.5 rpy=0 0 0
- joint left_front_wheel_joint: limit effort=10 velocity=3 -> effort=10 velocity=10
- joint left_steer_joint: limit lower=-0.69 upper=0.5 effort=10 velocity=3 -> lower=-0.523 upper=0.47 effort=10 velocity=3; origin xyz=1.8 -0.5 -0.25 rpy=0 0 0 -> xyz=1.8 -0.6 -0.25 rpy=0 0 0
- joint right_front_wheel_joint: limit effort=10 velocity=3 -> effort=10 velocity=10
- joint right_steer_joint: limit lower=-0.5 upper=0.69 effort=10 velocity=3 -> lower=-0.47 upper=0.523 effort=10 velocity=3; origin xyz=1.8 0.5 -0.25 rpy=0 0 0 -> xyz=1.8 0.6 -0.25 rpy=0 0 0
